File: KiCad/ardSpaceMouse/ardSpaceMouse.kicad_pcb (KiCad board)
At the start: 2 copper layers, 60.3 x 38.1 mm, 5 parts, among them SW1 SW_Push, SW2 SW_Push, SW3 SW_Push, U1 Sparkfun_Pro_Micro, U2 JOYSTICKPTH_my

Commit message: scad updates
Parts:
- removed U1: Sparkfun_Pro_Micro, My_Arduino2:Sparkfun_Pro_Micro_large
- removed U2: JOYSTICKPTH_my, SparkFun_Electromechanical:JOYSTICK_large
- added J1: 3-pin_button+2xGND_header, My_Headers:3-pin_button+2xGND_header_large, F.Cu at (71.3, 42.5)
- added J2: 3-pin_button+2xGND_header, My_Headers:3-pin_button+2xGND_header_large, F.Cu at (86.4, 43.2)
- added J3: 3-pin_button+2xGND_header, My_Headers:3-pin_button+2xGND_header_large, F.Cu at (73.6, 79.7)
- added REF**: MountingHole_3.2mm_M3, MountingHole:MountingHole_3.2mm_M3, F.Cu at (73.7, 74.8)
- added REF**: MountingHole_3.2mm_M3, MountingHole:MountingHole_3.2mm_M3, F.Cu at (73.7, 89.5)
- SW1, SW2: footprint My_Misc:SW_PUSH_6mm_large -> My_Misc:SW_PUSH-12mm_large
- moved SW1 99.6 mm to (66.6, 47.6)
- moved SW3 75.1 mm to (76.8, 84.5)
- moved SW2 70.1 mm to (94.8, 48.2)
Routing:
- net GND: track 189.8 -> 43.9 mm
- net X: track 69.6 -> 0.00 mm
- net Net-(U1-Pad14): track 66.1 -> 0.00 mm
- net VCC: track 43.6 -> 0.00 mm
- net Net-(J1-Pad1): track 28.8 -> 17.2 mm
- net Net-(J3-Pad1): track 16.0 -> 6.37 mm
- net Net-(J2-Pad1): track 21.1 -> 12.5 mm
- net Y: track 8.52 -> 0.00 mm
Other:
- board size 60.3 x 38.1 mm -> 45.7 x 61.6 mm
- board text removed: "ardSpaceMouse Jon Sagebrand github.com/ardSpaceMouse"

Commit message: OrbioSpaceMouse
Parts:
- added REF**: MountingHole_3.2mm_M3, MountingHole:MountingHole_3.2mm_M3, F.Cu at (88.3, 36.2)
- added REF**: MountingHole_3.2mm_M3, MountingHole:MountingHole_3.2mm_M3, F.Cu at (60.3, 54.6)
- added REF**: MountingHole_3.2mm_M3, MountingHole:MountingHole_3.2mm_M3, F.Cu at (60.3, 35.6)
- added REF**: MountingHole_3.2mm_M3, MountingHole:MountingHole_3.2mm_M3, F.Cu at (88.3, 55.2)
- moved J3 49.8 mm to (107.9, 43.5)
- moved REF** 49.8 mm to (108.0, 38.7)
- moved REF** 49.8 mm to (108.0, 53.4)
- moved SW3 49.8 mm to (111.1, 48.3)
Other:
- board size 45.7 x 61.6 mm -> 61.4 x 27.2 mm
Changed lines of the file:
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@@
   )
   (footprint "MountingHole:MountingHole_3.2mm_M3" (layer "F.Cu")
-    (at 73.66 74.803)
+    (at 107.95 38.663)
     (descr "Mounting Hole 3.2mm, no annular, M3")
     (tags "mounting hole 3.2mm no annular m3")
@@
   )
   (footprint "My_Headers:3-pin_button+2xGND_header_large" (layer "F.Cu")
-    (at 73.585 79.665)
+    (at 107.875 43.525)
     (descr "Through hole straight pin header, 1x03, 2.54mm pitch, single row")
     (tags "Through hole pin header THT 1x03 2.54mm single row")
@@
       (net 1 "GND") (pinfunction "GND2") (pintype "power_in"))
     (model "${KICAD6_3DMODEL_DIR}/Connector_PinHeader_2.54mm.3dshapes/PinHeader_1x03_P2.54mm_Vertical.wrl"
-      (offset (xyz 0 0 0))
+      (offset (xyz 0 0 -1.905))
       (scale (xyz 1 1 1))
-      (rotate (xyz 0 0 0))
-    )
+      (rotate (xyz 0 180 0))
+    )
+  )
+  (footprint "MountingHole:MountingHole_3.2mm_M3" (layer "F.Cu")
+    (at 88.265 36.195)
+    (descr "Mounting Hole 3.2mm, no annular, M3")
+    (tags "mounting hole 3.2mm no annular m3")
+    (attr exclude_from_pos_files exclude_from_bom)
+    (fp_text reference "REF**" (at 0 -4.2) (layer "F.SilkS")
+      (effects (font (size 1 1) (thickness 0.15)))
+    )
+    (fp_text value "MountingHole_3.2mm_M3" (at 0 4.2) (layer "F.Fab") hide
+      (effects (font (size 1 1) (thickness 0.15)))
+    )
+    (fp_text user "${REFERENCE}" (at 0.3 0) (layer "F.Fab")
+      (effects (font (size 1 1) (thickness 0.15)))
+    )
+    (fp_circle (center 0 0) (end 3.2 0) (layer "Cmts.User") (width 0.15) (fill none))
+    (fp_circle (center 0 0) (end 3.45 0) (layer "F.CrtYd") (width 0.05) (fill none))
+    (pad "" np_thru_hole circle (at 0 0) (size 3.2 3.2) (drill 3.2) (layers *.Cu *.Mask))
   )
   (footprint "My_Headers:3-pin_button+2xGND_header_large" (layer "F.Cu")
@@
   )
   (footprint "My_Misc:SW_PUSH_6mm_large" (layer "F.Cu")
-    (at 76.835 84.455 180)
+    (at 111.125 48.315 180)
     (descr "https://www.omron.com/ecb/products/pdf/en-b3f.pdf")
     (tags "tact sw push 6mm")
@@
     )
   )
+  (footprint "MountingHole:MountingHole_3.2mm_M3" (layer "F.Cu")
+    (at 60.325 54.61)
+    (descr "Mounting Hole 3.2mm, no annular, M3")
+    (tags "mounting hole 3.2mm no annular m3")
+    (attr exclude_from_pos_files exclude_from_bom)
+    (fp_text reference "REF**" (at 0 -4.2) (layer "F.SilkS")
+      (effects (font (size 1 1) (thickness 0.15)))
+    )
+    (fp_text value "MountingHole_3.2mm_M3" (at 0 4.2) (layer "F.Fab") hide
+      (effects (font (size 1 1) (thickness 0.15)))
+    )
+    (fp_text user "${REFERENCE}" (at 0.3 0) (layer "F.Fab")
+      (effects (font (size 1 1) (thickness 0.15)))
+    )
+    (fp_circle (center 0 0) (end 3.2 0) (layer "Cmts.User") (width 0.15) (fill none))
+    (fp_circle (center 0 0) (end 3.45 0) (layer "F.CrtYd") (width 0.05) (fill none))
+    (pad "" np_thru_hole circle (at 0 0) (size 3.2 3.2) (drill 3.2) (layers *.Cu *.Mask))
+  )
+  (footprint "MountingHole:MountingHole_3.2mm_M3" (layer "F.Cu")
+    (at 60.325 35.56)
+    (descr "Mounting Hole 3.2mm, no annular, M3")
+    (tags "mounting hole 3.2mm no annular m3")
+    (attr exclude_from_pos_files exclude_from_bom)
+    (fp_text reference "REF**" (at 0 -4.2) (layer "F.SilkS")
+      (effects (font (size 1 1) (thickness 0.15)))
+    )
+    (fp_text value "MountingHole_3.2mm_M3" (at 0 4.2) (layer "F.Fab") hide
+      (effects (font (size 1 1) (thickness 0.15)))
+    )
+    (fp_text user "${REFERENCE}" (at 0.3 0) (layer "F.Fab")
+      (effects (font (size 1 1) (thickness 0.15)))
+    )
+    (fp_circle (center 0 0) (end 3.2 0) (layer "Cmts.User") (width 0.15) (fill none))
+    (fp_circle (center 0 0) (end 3.45 0) (layer "F.CrtYd") (width 0.05) (fill none))
+    (pad "" np_thru_hole circle (at 0 0) (size 3.2 3.2) (drill 3.2) (layers *.Cu *.Mask))
+  )
   (footprint "My_Misc:SW_PUSH-12mm_large" (layer "F.Cu")
     (at 94.755995 48.205009 180)
@@
   )
   (footprint "MountingHole:MountingHole_3.2mm_M3" (layer "F.Cu")
-    (at 73.66 89.535)
+    (at 107.95 53.395)
     (descr "Mounting Hole 3.2mm, no annular, M3")
     (tags "mounting hole 3.2mm no annular m3")
@@
     (fp_circle (center 0 0) (end 3.45 0) (layer "F.CrtYd") (width 0.05) (fill none))
     (pad "" np_thru_hole circle locked (at 0 0) (size 3.2 3.2) (drill 3.2) (layers *.Cu *.Mask))
+  )
+  (footprint "MountingHole:MountingHole_3.2mm_M3" (layer "F.Cu")
+    (at 88.265 55.245)
+    (descr "Mounting Hole 3.2mm, no annular, M3")
+    (tags "mounting hole 3.2mm no annular m3")
+    (attr exclude_from_pos_files exclude_from_bom)
+    (fp_text reference "REF**" (at 0 -4.2) (layer "F.SilkS")
+      (effects (font (size 1 1) (thickness 0.15)))
+    )
+    (fp_text value "MountingHole_3.2mm_M3" (at 0 4.2) (layer "F.Fab") hide
+      (effects (font (size 1 1) (thickness 0.15)))
+    )
+    (fp_text user "${REFERENCE}" (at 0.3 0) (layer "F.Fab")
+      (effects (font (size 1 1) (thickness 0.15)))
+    )
+    (fp_circle (center 0 0) (end 3.2 0) (layer "Cmts.User") (width 0.15) (fill none))
+    (fp_circle (center 0 0) (end 3.45 0) (layer "F.CrtYd") (width 0.05) (fill none))
+    (pad "" np_thru_hole circle (at 0 0) (size 3.2 3.2) (drill 3.2) (layers *.Cu *.Mask))
   )
   (footprint "My_Headers:3-pin_button+2xGND_header_large" (layer "F.Cu")
@@
   (gr_line (start 62.39 31.755) (end 58.58 31.755) (layer "Edge.Cuts") (width 0.1))
   (gr_line (start 51.595 38.105) (end 51.595 52.075) (layer "Edge.Cuts") (width 0.1))
-  (gr_line (start 68.58 86.36) (end 71.12 93.345) (layer "Edge.Cuts") (width 0.1))
-  (gr_line (start 76.2 71.12) (end 71.12 71.12) (layer "Edge.Cuts") (width 0.1))
-  (gr_line (start 78.74 86.36) (end 78.74 78.105) (layer "Edge.Cuts") (width 0.1))
+  (gr_line (start 102.87 50.22) (end 105.41 57.205) (layer "Edge.Cuts") (width 0.1))
+  (gr_line (start 110.49 34.98) (end 105.41 34.98) (layer "Edge.Cuts") (width 0.1))
+  (gr_line (start 113.03 50.22) (end 113.03 41.965) (layer "Edge.Cuts") (width 0.1))
   (gr_line (start 97.295995 52.015009) (end 97.295995 39.315009) (layer "Edge.Cuts") (width 0.1))
-  (gr_line (start 71.12 93.345) (end 76.2 93.345) (layer "Edge.Cuts") (width 0.1))
-  (gr_line (start 78.74 78.105) (end 76.2 71.12) (layer "Edge.Cuts") (width 0.1))
+  (gr_line (start 105.41 57.205) (end 110.49 57.205) (layer "Edge.Cuts") (width 0.1))
+  (gr_line (start 113.03 41.965) (end 110.49 34.98) (layer "Edge.Cuts") (width 0.1))
   (gr_line (start 51.595 52.075) (end 58.58 58.425) (layer "Edge.Cuts") (width 0.1))
-  (gr_line (start 76.2 93.345) (end 78.74 86.36) (layer "Edge.Cuts") (width 0.1))
+  (gr_line (start 110.49 57.205) (end 113.03 50.22) (layer "Edge.Cuts") (width 0.1))
   (gr_line (start 73.82 40.645) (end 62.39 31.755) (layer "Edge.Cuts") (width 0.1))
-  (gr_line (start 71.12 71.12) (end 68.58 78.105) (layer "Edge.Cuts") (width 0.1))
+  (gr_line (start 105.41 34.98) (end 102.87 41.965) (layer "Edge.Cuts") (width 0.1))
   (gr_line (start 97.295995 39.315009) (end 89.675995 32.330009) (layer "Edge.Cuts") (width 0.1))
   (gr_line (start 87.135995 59.000009) (end 89.675995 59.000009) (layer "Edge.Cuts") (width 0.1))
   (gr_line (start 89.675995 32.330009) (end 87.135995 32.330009) (layer "Edge.Cuts") (width 0.1))
   (gr_line (start 58.58 31.755) (end 51.595 38.105) (layer "Edge.Cuts") (width 0.1))
-  (gr_line (start 68.58 78.105) (end 68.58 86.36) (layer "Edge.Cuts") (width 0.1))
+  (gr_line (start 102.87 41.965) (end 102.87 50.22) (layer "Edge.Cuts") (width 0.1))
   (segment (start 94.755995 48.205009) (end 82.055995 48.205009) (width 0.762) (layer "B.Cu") (net 1))
   (segment (start 71.28 47.54) (end 71.28 45.09) (width 0.762) (layer "B.Cu") (net 1))
-  (segment (start 73.585 82.205) (end 73.585 84.38) (width 0.762) (layer "B.Cu") (net 1))
+  (segment (start 107.875 46.065) (end 107.875 48.24) (width 0.762) (layer "B.Cu") (net 1))
   (segment (start 54.065 47.585) (end 71.325 47.585) (width 0.762) (layer "B.Cu") (net 1))
   (segment (start 71.325 47.585) (end 71.28 47.54) (width 0.762) (layer "B.Cu") (net 1))
-  (segment (start 70.335 84.455) (end 76.835 84.455) (width 0.762) (layer "B.Cu") (net 1))
-  (segment (start 73.585 84.38) (end 73.66 84.455) (width 0.762) (layer "B.Cu") (net 1))
+  (segment (start 104.625 48.315) (end 111.125 48.315) (width 0.762) (layer "B.Cu") (net 1))
+  (segment (start 107.875 48.24) (end 107.95 48.315) (width 0.762) (layer "B.Cu") (net 1))
   (segment (start 86.359995 45.806009) (end 86.500995 45.665009) (width 0.762) (layer "B.Cu") (net 1))
   (segment (start 86.359995 48.260009) (end 86.359995 45.806009) (width 0.762) (layer "B.Cu") (net 1))
@@
   (segment (start 82.255995 43.205009) (end 94.675995 43.205009) (width 0.762) (layer "B.Cu") (net 3))
   (segment (start 94.675995 43.205009) (end 94.755995 43.125009) (width 0.762) (layer "B.Cu") (net 3))
-  (segment (start 76.835 79.955) (end 70.54 79.955) (width 0.762) (layer "B.Cu") (net 4))
-  (segment (start 70.54 79.955) (end 70.485 80.01) (width 0.762) (layer "B.Cu") (net 4))
+  (segment (start 111.125 43.815) (end 104.83 43.815) (width 0.762) (layer "B.Cu") (net 4))
+  (segment (start 104.83 43.815) (end 104.775 43.87) (width 0.762) (layer "B.Cu") (net 4))
   (zone (net 0) (net_name "") (layer "B.Cu") (hatch edge 0.508)
     (connect_pads (clearance 0.508))
@@
     (polygon
       (pts
-        (xy 80.01 94.615)
-        (xy 67.31 94.615)
-        (xy 67.31 69.85)
-        (xy 80.01 69.85)
+        (xy 114.3 58.475)
+        (xy 101.6 58.475)
+        (xy 101.6 33.71)
+        (xy 114.3 33.71)
       )
     )
@@
     (polygon
       (pts
-        (xy 79.375 93.98)
-        (xy 67.945 93.98)
-        (xy 67.945 70.485)
-        (xy 79.375 70.485)
+        (xy 113.665 57.84)
+        (xy 102.235 57.84)
+        (xy 102.235 34.345)
+        (xy 113.665 34.345)
       )
     )
