File: KiCad/OrbionSpaceMouse_HW-2.5_FW_0.26.5/OrbionSpaceMouse_HW-2.5_FW_0.26.5.kicad_sch (KiCad schematic)
At the start: 9 parts

Commit message: orbion schematics
Parts:
- D?: value (none) -> NeoPixel_THT
- SW?: value (none) -> SW_Push
- U?: value (none) -> KY-023_JoyStick
- U?: value (none) -> KY-040_Rotary_Encoder
- U?: value (none) -> SSD1306_I2C_display
- U?: value (none) -> Sparkfun_Pro_Micro; footprint (none) -> Arduino:Sparkfun_Pro_Micro
Connections:
- net rst-brown: now reaches D?.3 (VDD), SW?.1, U?.2 (VCC), U?.22 (RST), U?.4 (VCC)
- net neop-orange: now reaches D?.4 (DIN), U?.16 (D15)
- net joy-purple: now reaches U?.20 (D21/A3), U?.3 (VRx)
- net joy-gray: now reaches U?.19 (D20/A2), U?.4 (VRy)
- net joy-white: now reaches U?.18 (D19/A1), U?.5 (SW)
- net but3-orange: now reaches SW?.2, U?.12 (~D9/A9)
- net enc-white: now reaches U?.1 (CLK), U?.7 (D4/A6)
- net enc-gray: now reaches U?.2 (DT), U?.8 (~D5)
- net disp-yellow: now reaches U?.3 (SCL), U?.6 (~D3)
- net disp-green: now reaches U?.4 (SDA), U?.5 (D2)
- net but1-blue: now reaches SW?.1, U?.10 (D7)
- net but2-purple: now reaches SW?.2, U?.11 (D8/A8)
Changed lines of the file:
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@@
     (stroke (width 0) (type default) (color 0 0 0 0))
+  )
+  (label "rst-brown" (at 162.56 64.77 0)
+    (effects (font (size 1.27 1.27)) (justify left bottom))
+  )
+  (label "but2-purple" (at 115.57 85.09 0)
+    (effects (font (size 1.27 1.27)) (justify left bottom))
+  )
+  (label "neop-orange" (at 162.56 80.01 0)
+    (effects (font (size 1.27 1.27)) (justify left bottom))
+  )
+  (label "joy-purple" (at 162.56 69.85 0)
+    (effects (font (size 1.27 1.27)) (justify left bottom))
+  )
+  (label "joy-white" (at 162.56 74.93 0)
+    (effects (font (size 1.27 1.27)) (justify left bottom))
+  )
+  (label "but3-orange" (at 115.57 87.63 0)
+    (effects (font (size 1.27 1.27)) (justify left bottom))
+  )
+  (label "enc-gray" (at 115.57 77.47 0)
+    (effects (font (size 1.27 1.27)) (justify left bottom))
+  )
+  (label "but1-blue" (at 115.57 82.55 0)
+    (effects (font (size 1.27 1.27)) (justify left bottom))
+  )
+  (label "enc-white" (at 115.57 74.93 0)
+    (effects (font (size 1.27 1.27)) (justify left bottom))
+  )
+  (label "disp-green" (at 115.57 69.85 0)
+    (effects (font (size 1.27 1.27)) (justify left bottom))
+  )
+  (label "joy-gray" (at 162.56 72.39 0)
+    (effects (font (size 1.27 1.27)) (justify left bottom))
+  )
+  (label "disp-yellow" (at 115.57 72.39 0)
+    (effects (font (size 1.27 1.27)) (justify left bottom))
   )
   (symbol (lib_id "LED:NeoPixel_THT") (at 205.74 121.92 0) (mirror x) (unit 1)
     (in_bom yes) (on_board yes) (fields_autoplaced)
     (property "Reference" "D?" (id 0) (at 193.5896 116.9628 0))
-    (property "Value" "" (id 1) (at 193.5896 119.4997 0))
+    (property "Value" "NeoPixel_THT" (id 1) (at 193.5896 119.4997 0))
     (property "Footprint" "" (id 2) (at 207.01 114.3 0)
       (effects (font (size 1.27 1.27)) (justify left top) hide)
@@
       (effects (font (size 1.27 1.27)) (justify left))
     )
-    (property "Value" "" (id 1) (at 224.2312 86.7922 0)
+    (property "Value" "KY-023_JoyStick" (id 1) (at 224.2312 86.7922 0)
       (effects (font (size 1.27 1.27)) (justify left))
     )
@@
     (in_bom yes) (on_board yes) (fields_autoplaced)
     (property "Reference" "U?" (id 0) (at 64.1349 70.0842 0))
-    (property "Value" "" (id 1) (at 64.135 67.31 0)
+    (property "Value" "KY-040_Rotary_Encoder" (id 1) (at 64.135 67.31 0)
       (effects (font (size 1.27 1.27)) hide)
     )
@@
     (in_bom yes) (on_board yes) (fields_autoplaced)
     (property "Reference" "U?" (id 0) (at 58.1025 34.5272 0))
-    (property "Value" "" (id 1) (at 58.1025 37.0641 0))
+    (property "Value" "SSD1306_I2C_display" (id 1) (at 58.1025 37.0641 0))
     (property "Footprint" "" (id 2) (at 65.405 36.83 0)
       (effects (font (size 1.27 1.27)) hide)
@@
       (effects (font (size 1.524 1.524)))
     )
-    (property "Value" "" (id 1) (at 144.78 55.9323 0)
+    (property "Value" "Sparkfun_Pro_Micro" (id 1) (at 144.78 55.9323 0)
       (effects (font (size 1.524 1.524)))
     )
-    (property "Footprint" "" (id 2) (at 144.78 91.44 0)
+    (property "Footprint" "Arduino:Sparkfun_Pro_Micro" (id 2) (at 144.78 91.44 0)
       (effects (font (size 1.524 1.524)) hide)
     )
@@
     (in_bom yes) (on_board yes) (fields_autoplaced)
     (property "Reference" "SW?" (id 0) (at 43.18 105.1392 0))
-    (property "Value" "" (id 1) (at 43.18 107.6761 0))
+    (property "Value" "SW_Push" (id 1) (at 43.18 107.6761 0))
     (property "Footprint" "" (id 2) (at 43.18 106.68 0)
       (effects (font (size 1.27 1.27)) hide)
